File: pre-amp-12AX7EH.sch (KiCad schematic (older format))
At the start: 19 parts, among them U1 12AX7EH

Commit message: feat: add values to components
Parts:
- removed C? (x2): 22n, symbol Device:C
- removed C?: 220u, symbol Device:C
- removed C?: C, symbol Device:C
- removed R?: 1k3, symbol Device:R
- removed R?: 100k, symbol Device:R
- removed R?: 1M, symbol Device:R
- removed R? (x3): R, symbol Device:R
- removed RV?: 1M, symbol Device:R_POT
- removed U1: 12AX7EH, Valve:Valve_Noval_P, symbol Valve:ECC83
- removed U? (x2): EL34, Valve:Valve_Octal, symbol Valve:EL34
- added C2: 220u, Resistor_THT:R_Axial_DIN0207_L6.3mm_D2.5mm_P7.62mm_Horizontal, symbol Device:C
- added C3, C5: 22n, symbol Device:C
- added C4: 220u, symbol Device:C
- added R5: 1M, Resistor_THT:R_Axial_DIN0207_L6.3mm_D2.5mm_P7.62mm_Horizontal, symbol Device:R
- added R6: 68k, Resistor_THT:R_Axial_DIN0207_L6.3mm_D2.5mm_P7.62mm_Horizontal, symbol Device:R
- added R7: 100k, symbol Device:R
- added R8: 4k, symbol Device:R
- added R9: 1M, symbol Device:R
- added RV1: 100k LOG, symbol Device:R_POT
- added RV2, RV3: 100k, symbol Device:R_POT
- added U1: 12AX7EH, Valve:Valve_Noval_P, symbol User~Valse:12AX7EH
- C1: value 220u -> 22n; Voltage rating 25 -> 600
- R1: footprint (none) -> Resistor_THT:R_Axial_DIN0207_L6.3mm_D2.5mm_P7.62mm_Horizontal; Power rating 0.25 -> 0.1
- R2: value 91k -> 68k; footprint (none) -> Resistor_THT:R_Axial_DIN0207_L6.3mm_D2.5mm_P7.62mm_Horizontal; Power rating 0.25 -> 0.1
- R3: value 1k3 -> 100k; Power rating 0.25 -> 1
- R4: value 100k -> 2k; footprint (none) -> Resistor_THT:R_Axial_DIN0207_L6.3mm_D2.5mm_P7.62mm_Horizontal; Power rating 2 -> (none)
Connections:
- net labels added: V+, V_IN, V_OUT
- net labels removed: +300V, +345V, Input
- wire segments 59 -> 46
Other:
- note removed: "OUTPUT TRANSFORMER\n"
